File: KiCad_Project/Audio_Amp_v1/05_Power_Amplifier.kicad_sch (KiCad schematic)
At the start: 0 parts

Commit message: Add power amplifier schematic, custom library, and initial components
Parts:
- added C1, C2, C3, C4, C5: 1u, symbol Device:C
- added C10, C17: 220u, symbol Device:C_Polarized_US
- added C11, C12, C13, C14: 220n, symbol Device:C
- added C15, C20, C21, C26, C27, C8: 1n, symbol Device:C
- added C16, C7, C9: 100n, symbol Device:C
- added C18, C19, C24, C25: 680n, symbol Device:C
- added C22, C23, C28, C29, C6: 10n, symbol Device:C
- added IC2: TPA3116D2DAD, SOP65P810X120-32N, symbol TPA3116D2DAD:TPA3116D2DAD
- added L1, L2, L3, L4: 10u, symbol Device:L
- added R1, R3, R4: 100k, symbol Device:R_US
- added R2: 20k, symbol Device:R_US
- added R5, R6, R7, R8, R9: 3.3R, symbol Device:R_US
Connections:
- new net: C3.2, IC2.7 (GVDD), R1.1
- new net: IC2.8 (GAIN/SLV), R1.2, R2.1
- new net: C23.1, R6.2
- new net: C2.2, IC2.5 (RINN)
- new net: C7.2, R5.2
- new net: C1.2, IC2.4 (RINP)
- new net: C12.1, IC2.26 (BSNR)
- new net: C12.2, IC2.27 (OUTNR), L2.2
- new net: C14.1, IC2.20 (BSNL)
- new net: C13.1, IC2.24 (BSPL)
- new net: C13.2, IC2.23 (OUTPL), L3.1
- new net: C29.2, R9.1
- new net: C4.1, IC2.10 (LINP)
- new net: C28.1, R8.2
- new net: C5.1, IC2.11 (LINN)
- new net: C11.2, IC2.29 (OUTPR), L1.1
- new net: C11.1, IC2.30 (BSPR)
- new net: C22.2, R7.1
- new net GNDA: C10.2, C14.2, C15.2, C16.2, C17.2, C18.2, C19.1, C20.2, C21.1, C22.1, C23.2, C24.2, C25.1, C26.2, C27.1, C28.2, C29.1, C3.1, C6.1, C7.1, C8.2, C9.2, IC2.1 (MODSEL), IC2.13 (AM2), IC2.14 (AM1), IC2.15 (AM0), IC2.21 (OUTNL), IC2.22 (GND_2), IC2.25 (GND_3), IC2.28 (GND_4), IC2.9 (GND_1), L4.2, R2.2, R3.2
- new net IN_N_LEFT: C5.2
- new net IN_N_RIGHT: C2.1
- new net IN_P_LEFT: C4.2
- new net IN_P_RIGHT: C1.1
- new net MUTE_LR: IC2.12 (MUTE), R3.1
- new net OUT_N_LEFT: C25.2, C27.2, L4.1, R9.2
- new net OUT_N_RIGHT: C19.2, C21.2, L2.1, R7.2
- new net OUT_P_LEFT: C24.1, C26.1, L3.2, R8.1
- new net OUT_P_RIGHT: C18.1, C20.1, L1.2, R6.1
- new net PVCC: C10.1, C15.1, C16.1, C17.1, C6.2, C8.1, C9.1, IC2.17 (AVCC), IC2.18 (PVCC_1), IC2.19 (PVCC_2), IC2.31 (PVCC_3), IC2.32 (PVCC_4), R4.1, R5.1
- new net /SD_LR: IC2.2 (SDZ), IC2.3 (FAULTZ), R4.2
- no-connect marks 0 -> 1
Other:
- note added: "4R"
- note added: "EMI C-RC SNUBBER"
- note added: "OUTPUT LC FILTER"
- note added: "PVCC DECOUPLING"

Commit message: Added some passive components and updated the Power amplifier schematic with footprints
Parts:
- C1, C2, C20, C21, C22, C23, C26, C27, C28, C29, C3, C4, C5, C6, C7: footprint (none) -> Capacitor_SMD:C_0603_1608Metric
- C10, C17: footprint (none) -> EEE-FK1H221GV:EEHZT1E561UV
- C11, C12, C13, C14, C15, C16, C8, C9: footprint (none) -> Capacitor_SMD:C_0805_2012Metric
- C18, C19, C24, C25: footprint (none) -> Capacitor_SMD:C_1206_3216Metric
- L1, L2, L3, L4: footprint (none) -> 7443341000:INDPM8479X720N
- R1, R2, R3, R4: footprint (none) -> Resistor_SMD:R_0603_1608Metric
- R5, R6, R7, R8, R9: footprint (none) -> Resistor_SMD:R_1206_3216Metric
Connections:
- net GNDA: now also IC2.33 (GND), L4.1; no longer L4.2
- net OUT_N_LEFT: now also L4.2; no longer L4.1
- net at C3.2, IC2.7 (GVDD), R1.1: now also IC2.6 (PLIMIT)

Commit message: Updated Power management section, Bluetooth receiver and connectors. Added some components footprints and 3D.
Connections:
- net IN_N_RIGHT is gone; now on net IN_COM: C2.1
- net GNDA: now also R3.1; no longer R3.2
- net IN_N_LEFT renamed IN_COM
- net MUTE_LR: no longer names the net of IC2.12 (MUTE)
- net MUTE_LR: now also R3.2; no longer R3.1
- net PVCC renamed +24V
- net /SD_LR: no longer names the net of IC2.2 (SDZ), IC2.3 (FAULTZ), R4.2
Other:
- note added: "Anti POP pin always connected to VDD"
- note added: "MUTE PIN actually pulled to gnda"
- moved on the sheet: R3

Commit message: Finished Schematic and started Layout
Parts:
- IC2: footprint SOP65P810X120-32N -> TPA3116D2DAD:SOP65P810X120-32N
Changed lines of the file:
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@@
 	)
 	(junction
+		(at 85.09 67.31)
+		(diameter 0)
+		(color 0 0 0 0)
+	)
+	(junction
 		(at 215.9 66.04)
 		(diameter 0)
@@
 	)
 	(junction
+		(at 109.22 39.37)
+		(diameter 0)
+		(color 0 0 0 0)
+	)
+	(junction
 		(at 67.31 107.95)
 		(diameter 0)
@@
 	(wire
 		(pts
-			(xy 109.22 36.83) (xy 109.22 41.91)
+			(xy 109.22 36.83) (xy 109.22 39.37)
 		)
 		(stroke
@@
 	(wire
 		(pts
+			(xy 82.55 67.31) (xy 85.09 67.31)
+		)
+		(stroke
+			(width 0)
+			(type default)
+		)
+	)
+	(wire
+		(pts
 			(xy 215.9 66.04) (xy 215.9 68.58)
 		)
@@
 	(wire
 		(pts
-			(xy 82.55 67.31) (xy 90.17 67.31)
-		)
-		(stroke
-			(width 0)
-			(type default)
-		)
-	)
-	(wire
-		(pts
 			(xy 135.89 41.91) (xy 135.89 71.12)
 		)
@@
 	(wire
 		(pts
+			(xy 109.22 39.37) (xy 109.22 41.91)
+		)
+		(stroke
+			(width 0)
+			(type default)
+		)
+	)
+	(wire
+		(pts
 			(xy 77.47 123.19) (xy 87.63 123.19)
 		)
@@
 	(wire
 		(pts
+			(xy 85.09 67.31) (xy 90.17 67.31)
+		)
+		(stroke
+			(width 0)
+			(type default)
+		)
+	)
+	(wire
+		(pts
 			(xy 110.49 52.07) (xy 100.33 52.07)
 		)
@@
 	(wire
 		(pts
+			(xy 106.68 39.37) (xy 109.22 39.37)
+		)
+		(stroke
+			(width 0)
+			(type default)
+		)
+	)
+	(wire
+		(pts
 			(xy 90.17 78.74) (xy 90.17 74.93)
 		)
@@
 	(wire
 		(pts
+			(xy 85.09 64.77) (xy 85.09 67.31)
+		)
+		(stroke
+			(width 0)
+			(type default)
+		)
+	)
+	(wire
+		(pts
 			(xy 85.09 115.57) (xy 67.31 115.57)
 		)
@@
 			)
 		)
-		(property "Footprint" "SOP65P810X120-32N"
+		(property "Footprint" "TPA3116D2DAD:SOP65P810X120-32N"
 			(at 127 187.63 0)
 			(hide yes)
@@
 	)
 	(symbol
+		(lib_id "power:PWR_FLAG")
+		(at 85.09 64.77 0)
+		(unit 1)
+		(body_style 1)
+		(exclude_from_sim no)
+		(in_bom yes)
+		(on_board yes)
+		(in_pos_files yes)
+		(dnp no)
+		(property "Reference" "#FLG03"
+			(at 85.09 62.865 0)
+			(hide yes)
+			(show_name no)
+			(do_not_autoplace no)
+			(effects
+				(font
+					(size 1.27 1.27)
+				)
+			)
+		)
+		(property "Value" "PWR_FLAG"
+			(at 91.186 62.992 0)
+			(show_name no)
+			(do_not_autoplace no)
+			(effects
+				(font
+					(size 1.27 1.27)
+				)
+			)
+		)
+		(property "Footprint" ""
+			(at 85.09 64.77 0)
+			(hide yes)
+			(show_name no)
+			(do_not_autoplace no)
+			(effects
+				(font
+					(size 1.27 1.27)
+				)
+			)
+		)
+		(property "Datasheet" ""
+			(at 85.09 64.77 0)
+			(hide yes)
+			(show_name no)
+			(do_not_autoplace no)
+			(effects
+				(font
+					(size 1.27 1.27)
+				)
+			)
+		)
+		(property "Description" "Special symbol for telling ERC where power comes from"
+			(at 85.09 64.77 0)
+			(hide yes)
+			(show_name no)
+			(do_not_autoplace no)
+			(effects
+				(font
+					(size 1.27 1.27)
+				)
+			)
+		)
+		(pin "1"
+		)
+		(instances
+			(project "Audio_Amp_v1"
+				(path "/d992164b-b1d0-4285-be2c-12a40c17e5cc/bcd969c5-e603-453f-8e84-f4a0a5ebae98"
+					(reference "#FLG03")
+					(unit 1)
+				)
+			)
+		)
+	)
+	(symbol
 		(lib_id "Device:C")
 		(at 66.04 48.26 180)
@@
 					(unit 1)
 				)
+			)
+		)
+	)
+	(symbol
+		(lib_id "power:PWR_FLAG")
+		(at 106.68 39.37 90)
+		(unit 1)
+		(body_style 1)
+		(exclude_from_sim no)
+		(in_bom yes)
+		(on_board yes)
+		(in_pos_files yes)
+		(dnp no)
+		(fields_autoplaced yes)
+		(property "Reference" "#FLG01"
+			(at 104.775 39.37 0)
+			(hide yes)
+			(show_name no)
+			(do_not_autoplace no)
+			(effects
+				(font
+					(size 1.27 1.27)
+				)
+			)
+		)
+		(property "Value" "PWR_FLAG"
+			(at 102.87 39.3699 90)
+			(show_name no)
+			(do_not_autoplace no)
+			(effects
+				(font
+					(size 1.27 1.27)
+				)
+				(justify left)
+			)
+		)
+		(property "Footprint" ""
+			(at 106.68 39.37 0)
+			(hide yes)
+			(show_name no)
+			(do_not_autoplace no)
+			(effects
+				(font
+					(size 1.27 1.27)
+				)
+			)
+		)
+		(property "Datasheet" ""
+			(at 106.68 39.37 0)
+			(hide yes)
+			(show_name no)
+			(do_not_autoplace no)
+			(effects
+				(font
+					(size 1.27 1.27)
+				)
+			)
+		)
+		(property "Description" "Special symbol for telling ERC where power comes from"
+			(at 106.68 39.37 0)
+			(hide yes)
+			(show_name no)
+			(do_not_autoplace no)
+			(effects
+				(font
+					(size 1.27 1.27)
+				)
+			)
+		)
+		(pin "1"
+		)
+		(instances
+			(project "Audio_Amp_v1"
+				(path "/d992164b-b1d0-4285-be2c-12a40c17e5cc/bcd969c5-e603-453f-8e84-f4a0a5ebae98"
+					(reference "#FLG01")
+					(unit 1)
+				)

Commit message: Layout Updated, finished routing
Connections:
- net GNDA: no longer C14.2, IC2.21 (OUTNL), L4.1
- new net: C14.2, IC2.21 (OUTNL), L4.1
Changed lines of the file:
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@@
-	)
-	(junction
-		(at 172.72 149.86)
-		(diameter 0)
-		(color 0 0 0 0)
 	)
 	(junction
@@
 		)
 		(stroke
-			(width 0)
-			(type default)
-		)
-	)
-	(wire
-		(pts
-			(xy 172.72 149.86) (xy 163.83 149.86)
-		)
-		(stroke
