File: KiCad_Project/Audio_Amp_v1/Audio_Amp_v1.kicad_pcb (KiCad board)
At the start: 2 copper layers, 100 x 75 mm, 71 parts, among them IC2 TPA3116D2DAD, IC3 BM64SPKS1MC2-0002AA, IC4 LMR33630ADDA, J1 TS-103-T-A, J2 1729128, J3 1729128, J4 PJ-102AH

Commit message: Continued Layout
Parts:
- added TP3: TestPoint, TestPoint:TestPoint_Pad_D2.0mm, F.Cu at (90.2, 101.2)
- added TP4: TestPoint, TestPoint:TestPoint_Pad_D2.0mm, F.Cu at (86.5, 101.2)
- moved J1 122.3 mm to (101.5, 129.8), turned to 0 degrees
- moved C17 120.1 mm to (115.8, 124.4)
- moved TP2 119.8 mm to (84.7, 128.5), turned to 180 degrees
- moved R10 117.8 mm to (88.5, 128.5), turned to 180 degrees
- moved C64 116.1 mm to (88.5, 126.8), turned to 0 degrees
- moved C31 107.9 mm to (97.7, 117.8), turned to 0 degrees
- moved C30 106.8 mm to (97.7, 116.2), turned to 0 degrees
- moved R11 102.2 mm to (97.0, 112.8), turned to -90 degrees
- moved TP1 102.1 mm to (101.5, 112.8), turned to 180 degrees
- moved R16 102.1 mm to (98.5, 112.8), turned to -90 degrees
- moved C25 100.0 mm to (144.5, 123.2), turned to -90 degrees
- moved J4 98.7 mm to (76.5, 98.8)
- moved R9 97.5 mm to (148.3, 126.2), turned to 180 degrees
- moved D1 97.0 mm to (92.2, 105.8), turned to 0 degrees
- moved R13 96.9 mm to (75.7, 105.2), turned to -90 degrees
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Routing:
- net Net-(IC2-OUTPR): track 0.00 -> 18.8 mm
- net Net-(IC2-OUTPL): track 0.00 -> 12.1 mm
- net Net-(IC2-OUTNR): track 0.00 -> 11.5 mm
- net OUT_N_RIGHT: track 0.00 -> 10.9 mm
- net OUT_P_RIGHT: track 0.00 -> 10.6 mm
- net OUT_P_LEFT: track 0.00 -> 10.3 mm
- net OUT_N_LEFT: track 0.00 -> 8.41 mm
- net Net-(IC2-BSNR): track 0.00 -> 6.17 mm
- net Net-(IC2-RINP): track 0.00 -> 5.40 mm
- net Net-(IC2-GAIN/SLV): track 0.00 -> 5.33 mm
- net Net-(IC2-FAULTZ): track 0.00 -> 4.82 mm
- net Net-(IC2-RINN): track 0.00 -> 4.31 mm
- net Net-(IC2-MUTE): track 0.00 -> 4.14 mm
- net Net-(IC2-BSPR): track 0.00 -> 3.43 mm
- net Net-(IC2-LINN): track 0.00 -> 3.12 mm
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Other:
- board size 100 x 75 mm -> 93.5 x 54.8 mm

Commit message: Layout Updated, finished routing
Parts:
- moved TP4 14.8 mm to (101.0, 104.0)
- moved TP2 7.57 mm to (92.2, 128.0)
- moved R10 3.65 mm to (85.2, 126.8), turned to 0 degrees
- moved J2 2.80 mm to (156.8, 97.7)
- moved C14 2.70 mm to (127.2, 112.5), turned to 90 degrees
- moved C20 2.52 mm to (146.8, 97.4)
- moved C21 2.52 mm to (146.8, 101.9)
- moved C22 2.52 mm to (148.5, 101.9)
- moved C23 2.52 mm to (148.5, 97.4)
- moved R6 2.52 mm to (148.2, 94.5)
- moved R7 2.52 mm to (148.2, 104.9)
- moved C1 2.50 mm to (110.3, 103.1)
- moved C10 2.50 mm to (117.0, 88.3), turned to -90 degrees
- moved C11 2.50 mm to (125.2, 104.8)
- moved C12 2.50 mm to (128.3, 106.9)
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Connections:
- C14 pad 2: GNDA -> Net-(IC2-OUTNL)
- IC2 pad 21: GNDA -> Net-(IC2-OUTNL)
- J1 pad 01: UART_TX -> UART_RX
- J1 pad 02: UART_RX -> UART_TX
- L4 pad 1: GNDA -> Net-(IC2-OUTNL)
Routing:
- net +24V: track 0.00 -> 107.2 mm, vias 0 -> 25
- net GNDA: track 1.47 -> 63.1 mm, vias 4 -> 63
- net +3.3V: track 36.0 -> 94.9 mm, vias 2 -> 15
- net IN_COM: track 0.00 -> 54.5 mm, vias 0 -> 2
- net IN_P_RIGHT: track 0.00 -> 45.2 mm
- net IN_P_LEFT: track 0.00 -> 39.0 mm
- net OUT_N_LEFT: track 8.41 -> 34.0 mm
- net OUT_N_RIGHT: track 10.9 -> 35.0 mm
- net OUT_P_RIGHT: track 10.6 -> 34.4 mm
- net OUT_P_LEFT: track 10.3 -> 34.0 mm
- net Net-(IC2-OUTNL): track 0.00 -> 21.3 mm
- net UART_TX: track 0.00 -> 15.3 mm, vias 0 -> 1
- net UART_RX: track 0.00 -> 11.8 mm, vias 0 -> 1
- net Net-(D1-A): track 0.00 -> 10.9 mm, vias 0 -> 2
- net /02_Bluetooth_Receiver/RST_N: track 0.00 -> 10.3 mm
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- added copper zone on B.Cu, net GNDA
Other:
- board size 93.5 x 54.8 mm -> 93.5 x 52.8 mm
